Commit message: add test

File: cartographer_ros/urdf/backpack_3d_lp.urdf (robot description, URDF)
Before this commit: robot cartographer_backpack_2d, 6 links, 5 joints
Links:
- added link laser_link
Joints:
- added joint laser_base_link_joint: type fixed, parent base_link, child laser_link, origin xyz=0 0 0 rpy=0 0 0
